File: RS-485-Interface-Unit.brd (EAGLE design)
At the start: 53.4 x 35.9 mm, 16 parts, among them IC1 B0505S, IC2 ADM2483, IC3 78L05Z, X1 RJ11CONNECTOR, X2 RJ11CONNECTOR

Commit message: Updated pcb
Parts:
- moved JP7 14.4 mm to (24.7, 32.7), turned to 180 degrees
- moved R11 11.9 mm to (43.3, 29.6), turned to 0 degrees
- moved JP6 7.68 mm to (29.2, 32.7), turned to 180 degrees
- moved C3 6.62 mm to (22.1, 32.7), turned to 90 degrees
- moved C4 5.88 mm to (17.9, 26.2), turned to 270 degrees
- moved IC3 4.74 mm to (18.4, 31.5), turned to 90 degrees
- moved C2 2.76 mm to (20.5, 26.2), turned to 270 degrees
- moved JP2 1.94 mm to (36.8, 32.9)
- moved C1 1.30 mm to (29.0, 18.3)
- moved R2 0.40 mm to (20.9, 19.2)
Routing:
- net +3V3: track 46.1 -> 3.87 mm, vias 3 -> 1
- net POWER_VALID: track 14.4 -> 11.3 mm
- net +12V: track 9.37 -> 6.90 mm
- net !RE: track 7.17 -> 5.41 mm
- net DE: track 6.65 -> 4.90 mm
- net UART_RX: track 11.2 -> 9.49 mm
- net VCCIO: track 13.5 -> 12.0 mm
- net GNDIO: track 25.2 -> 24.3 mm
- net GND: track 68.7 -> 69.4 mm
- net UART_TX: track 6.12 -> 5.42 mm
Other:
- board size 53.4 x 35.9 mm -> 53.4 x 30.4 mm

Commit message: Board tracing done
Parts:
- JP1: value (none) -> TERM
- moved R11 1.57 mm to (44.0, 31.0)
- moved JP2 1.12 mm to (37.8, 32.4)
- moved C2 0.81 mm to (20.6, 27.0)
- moved JP6 0.30 mm to (29.2, 32.4)
- moved JP7 0.30 mm to (24.7, 32.4)
Routing:
- net GND: track 69.4 -> 75.0 mm, vias 1 -> 0
- net VCCIO: track 12.0 -> 13.9 mm
- net +3V3: track 3.87 -> 5.42 mm, vias 1 -> 0
- net UART_RX: track 9.49 -> 8.32 mm
- net UART_TX: track 5.42 -> 6.40 mm
- net !RE: track 5.41 -> 4.50 mm
- net GNDIO: track 24.3 -> 25.1 mm
- net POWER_VALID: track 11.3 -> 10.6 mm
- net +5V: track 17.5 -> 17.0 mm, vias 0 -> 2
Other:
- board size 53.4 x 30.4 mm -> 53 x 30 mm
- board text added: "!RE! RX"
- board text added: "+12"
- board text added: "+3.3"
- board text added: "DE GND"
- board text added: "GND"
- board text added: "PV TX"
- board text added: "TERM"
